Commit message: 0721

File: livelybot_HPM_control/legged_gym/resources/robots/pai_12dof/urdf/pai_12dof.urdf (robot description, URDF)
Before this commit: robot pai_12dof_v2_0312, 13 links, 12 joints
Links:
- link base_link: geometry collision box size=0.08 0.08 0.08; visual mesh filename=../meshes/base_link.STL
- link l_ankle_pitch_link: geometry collision box size=0.01 0.01 0.01; visual mesh filename=../meshes/l_ankle_pitch_link.STL
- link l_ankle_roll_link: geometry collision mesh filename=../meshes/l_ankle_roll_link.STL; visual mesh filename=../meshes/l_ankle_roll_link.STL
- link l_calf_link: geometry collision box size=0.01 0.01 0.01; visual mesh filename=../meshes/l_calf_link.STL
- link l_hip_roll_link: geometry collision box size=0.01 0.01 0.01; visual mesh filename=../meshes/l_hip_roll_link.STL
- link l_hip_yaw_link: geometry collision box size=0.01 0.01 0.01; visual mesh filename=../meshes/l_hip_yaw_link.STL
- link l_thigh_link: geometry collision box size=0.01 0.01 0.01; visual mesh filename=../meshes/l_thigh_link.STL
- link r_ankle_pitch_link: geometry collision box size=0.01 0.01 0.01; visual mesh filename=../meshes/r_ankle_pitch_link.STL
- link r_ankle_roll_link: geometry collision mesh filename=../meshes/r_ankle_roll_link.STL; visual mesh filename=../meshes/r_ankle_roll_link.STL
- link r_calf_link: geometry collision box size=0.01 0.01 0.01; visual mesh filename=../meshes/r_calf_link.STL
- link r_hip_roll_link: geometry collision box size=0.01 0.01 0.01; visual mesh filename=../meshes/r_hip_roll_link.STL
- link r_hip_yaw_link: geometry collision box size=0.01 0.01 0.01; visual mesh filename=../meshes/r_hip_yaw_link.STL
- link r_thigh_link: geometry collision box size=0.01 0.01 0.01; visual mesh filename=../meshes/r_thigh_link.STL
