Commit message: 20240729_update

File: livelybot_GYM_control/assets/urdf/pai_12dof/urdf/pai_12dof.urdf (robot description, URDF)
Before this commit: robot pai_12dof_v2_0312, 13 links, 12 joints
Joints:
- joint left_knee_joint: axis 0 -1 0 -> 0 1 0; limit lower=-2.0 upper=0.0 effort=21 velocity=21 -> lower=0.0 upper=2.0 effort=21 velocity=21
- joint right_ankle_pitch_joint: axis 0 -1 0 -> 0 1 0; limit lower=-0.6 upper=0.7 effort=21 velocity=21 -> lower=-0.7 upper=0.6 effort=21 velocity=21
- joint right_hip_pitch_joint: axis 0 -1 0 -> 0 1 0; limit lower=-0.48 upper=1.57 effort=21 velocity=21 -> lower=-1.57 upper=0.48 effort=21 velocity=21

File: src/pai_12dof/urdf/pai_12dof.urdf (robot description, URDF)
Before this commit: robot pai_12dof_v2_0312, 13 links, 12 joints
Joints:
- joint left_knee_joint: axis 0 -1 0 -> 0 1 0; limit lower=-2.0 upper=0.0 effort=21 velocity=21 -> lower=0.0 upper=2.0 effort=21 velocity=21
- joint right_ankle_pitch_joint: axis 0 -1 0 -> 0 1 0; limit lower=-0.6 upper=0.7 effort=21 velocity=21 -> lower=-0.7 upper=0.6 effort=21 velocity=21
- joint right_hip_pitch_joint: axis 0 -1 0 -> 0 1 0; limit lower=-0.48 upper=1.57 effort=21 velocity=21 -> lower=-1.57 upper=0.48 effort=21 velocity=21
